File: pcb/200280.kicad_pcb (KiCad board)
At the start: 2 copper layers, 125 x 25 mm, 19 parts, among them J1 ScrewTerms, Q1 2N3904, Q2 2N3904, Q3 2N3904, U1 SN74AVC8T245PW, U2 XIAO-ESP32-S3-SMD, U3 OKI-78SR-5/1.5-W36-C

Commit message: final PCB design as purchased rev A
Parts:
- removed Q3: 2N3904, Package_TO_SOT_SMD:SOT-23-3
- added Q4: MMBT3904, Package_TO_SOT_SMD:SOT-23-3, F.Cu at (123.9, 78.5)
- added R7: 120R, Resistor_SMD:R_0603_1608Metric, F.Cu at (146.3, 94.1)
- C1: footprint Capacitor_SMD:C_1206_3216Metric -> Capacitor_SMD:C_0603_1608Metric
- J1: footprint Connector_Phoenix_MC:PhoenixContact_MCV_1,5_10-GF-3.5_1x10_P3.50mm_Vertical_ThreadedFlange -> GM_Connector_PhoenixContact:phoenix_contact_1984691
- Q1: value 2N3904 -> MMBT3904
- Q2: value 2N3904 -> SI2304BDS-T1-GE3; footprint Package_TO_SOT_SMD:SOT-23-3 -> Package_TO_SOT_SMD:SOT-23
- R1, R2, R3, R4, R5, R6: footprint Resistor_SMD:R_1206_3216Metric -> Resistor_SMD:R_0603_1608Metric
- moved Q2 17.9 mm to (139.3, 92.2), turned to 180 degrees
- moved R3 5.90 mm to (129.0, 81.7), turned to -90 degrees
- moved U3 4.91 mm to (106.5, 81.0)
- moved Q1 3.60 mm to (128.1, 78.5)
- moved R1 3.35 mm to (125.7, 81.7), turned to -90 degrees
- moved C1 3.15 mm to (130.7, 81.7), turned to -90 degrees
- moved H1 2.50 mm to (60.0, 87.5)
- moved H4 2.50 mm to (175.0, 87.5)
- moved R2 2.11 mm to (127.2, 81.7), turned to -90 degrees
- moved R4 1.83 mm to (132.4, 81.7), turned to 90 degrees
- moved D1 1.45 mm to (124.2, 81.9)
- moved R6 0.83 mm to (122.7, 81.8)
- moved J1 0.79 mm to (67.2, 80.2)
- moved C3 0.68 mm to (139.4, 80.0)
- moved C2 0.38 mm to (142.4, 80.0)
Connections:
- C1 pad 1: Net-(Q2-C) -> Net-(Q1-C)
- Q1 pad 1: GND -> Net-(Q1-B)
- Q1 pad 2: Net-(D1-K) -> GND
- Q2 pad 1: GND -> Net-(Q2-G)
- Q2 pad 2: Net-(Q2-B) -> GND
- Q2 pad 3: Net-(Q2-C) -> /WallButton
- R1 pad 1: Net-(Q1-C) -> Net-(Q4-C)
- R1 pad 2: Net-(Q2-B) -> Net-(Q1-B)
- R2 pad 1: Net-(Q1-C) -> Net-(Q4-C)
- R3 pad 1: Net-(Q2-C) -> Net-(Q1-C)
- R4 pad 2: Net-(Q2-C) -> Net-(Q1-C)
Routing:
- net +3V3: track 41.3 -> 61.3 mm
- net Net-(Q1-B): track 0.00 -> 9.70 mm
- net Net-(Q2-C): track 7.38 -> 0.00 mm
- net Net-(Q2-G): track 0.00 -> 6.11 mm
- net /WallButton: track 84.5 -> 78.8 mm
- net /WallButtonSimulation: track 8.85 -> 3.70 mm
- net +5V: track 80.8 -> 85.5 mm, vias 3 -> 4
- net /PowerIn: track 22.2 -> 17.6 mm
- net Net-(Q4-C): track 0.00 -> 4.15 mm
- net Net-(Q2-B): track 4.14 -> 0.00 mm
- net /Obstruction: track 37.5 -> 34.1 mm
- net /Relay3_: track 69.9 -> 73.1 mm
- net /ObstructionObserved: track 2.95 -> 5.60 mm
- net GND: track 16.0 -> 18.6 mm, vias 12 -> 14
- net /Relay2_: track 67.0 -> 69.1 mm
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Other:
- board size 125 x 25 mm -> 175 x 25 mm
- board text added: "Button Out"
- board text added: "Closed"
- board text added: "GND"
- board text added: "Light"
- board text added: "Obstruction"
- board text added: "Open"
- board text added: "PowerIn DC"
- board text added: "Relay2"
- board text added: "Relay3"
