File: pcb/200280.kicad_sch (KiCad schematic)
At the start: 19 parts, among them J1 ScrewTerms, Q1 2N3904, Q2 2N3904, Q3 2N3904, U1 SN74AVC8T245PW, U2 XIAO-ESP32-S3-SMD, U3 OKI-78SR-5/1.5-W36-C

Commit message: final PCB design as purchased rev A
Parts:
- removed Q1, Q2: 2N3904, Package_TO_SOT_THT:TO-92_Inline, symbol Transistor_BJT:2N3904
- removed Q3: 2N3904, Package_TO_SOT_SMD:SOT-23-3, symbol Transistor_BJT:2N3904
- added Q1, Q4: MMBT3904, Package_TO_SOT_SMD:SOT-23-3, symbol Device:Q_NPN_BEC
- added Q2: SI2304BDS-T1-GE3, Package_TO_SOT_SMD:SOT-23, symbol Device:Q_NMOS_GSD
- added R7: 120R, Resistor_SMD:R_0603_1608Metric, symbol Device:R_US
- C1: footprint Capacitor_SMD:C_1206_3216Metric -> Capacitor_SMD:C_0603_1608Metric
- J1: footprint Connector_Phoenix_MC:PhoenixContact_MC_1,5_10-GF-3.5_1x10_P3.50mm_Horizontal_ThreadedFlange_MountHole -> GM_Connector_PhoenixContact:phoenix_contact_1984691
- R1, R2, R3, R4, R5, R6: footprint Resistor_SMD:R_1206_3216Metric -> Resistor_SMD:R_0603_1608Metric
Connections:
- net GND: now also Q1.2 (E), Q2.2 (S), Q4.2 (E)
- net WallButton: now also Q2.3 (D)
- net WallButtonSimulation: now also R7.1
- net at C1.1, R3.1, R4.2: now also Q1.3 (C)
- net at D1.1 (K): now also Q4.1 (B)
- net at R1.1, R2.1: now also Q4.3 (C)
- net at R1.2: now also Q1.1 (B)
- new net: Q2.1 (G), R7.2
