File: pcb/200280rB.kicad_pcb (KiCad board)
At the start: 2 copper layers, 175 x 25 mm, 24 parts, among them J1 ScrewTerms, Q2 SI2304BDS-T1-GE3, Q3 SI2304BDS-T1-GE3, U1 SN74AVC8T245PW, U2 XIAO-ESP32-S3-SMD, U3 OKI-78SR-5/1.5-W36-C

Commit message: as purchased revision B
Parts:
- removed the C1 at (145.5, 78.5)
- removed D2, D3: MMBD4448HTS, Package_TO_SOT_SMD:SOT-523
- added C3: 1uF, Capacitor_SMD:C_0603_1608Metric, F.Cu at (126.5, 83.5)
- added Q1: MMBT3904, Package_TO_SOT_SMD:SOT-23-3, F.Cu at (122.5, 79.5)
- added Q2: MMBT3904, Package_TO_SOT_SMD:SOT-23-3, F.Cu at (127.5, 79.5)
- added R6: 680R, Resistor_SMD:R_0603_1608Metric, F.Cu at (129.5, 83.5)
- D1: value MMBD4448HTS -> 5.1V; footprint Package_TO_SOT_SMD:SOT-523 -> Diode_SMD:D_SOD-323_HandSoldering
- R1: value 100K -> 10K
- R2: value DNP -> 1K
- R3: value 100K -> 2K
- R4: value 680R -> 20K
- R5: value 680R -> 100K
- moved R3 22.8 mm to (123.0, 83.5), turned to -90 degrees
- moved R4 22.0 mm to (124.5, 83.5), turned to 90 degrees
- moved D1 9.01 mm to (121.0, 84.0), turned to -90 degrees
- moved R2 7.59 mm to (119.0, 83.5), turned to 90 degrees
- moved R5 7.15 mm to (128.0, 83.5)
- moved R1 5.85 mm to (117.5, 83.5), turned to -90 degrees
- renumbered C3 to C1, H4 to H2, Q2 to Q4, R7 to R10, R10 to R7, R9 to R8, R8 to R9, U3 to U1, U1 to U2, U2 to U3
Connections:
- net /Relay2_ renamed /Relay2_Motor_Closing
- net /Relay2__3V renamed /Relay2_Motor_Closing_3V
- net /Relay3_ renamed /Relay3_Motor_Opening
- net /Relay3__3V renamed /Relay3_Motor_Opening_3V
- D1 pad 1: Net-(D1-A) -> Net-(D1-K)
- D1 pad 2: Net-(D1-K) -> GND
- J1 pad 2: /Return? -> unconnected-(J1-Pin_2-Pad2)
- R1 pad 1: /Obstruction_5V -> Net-(D1-K)
- R1 pad 2: +5V -> /Obstruction
- R2 pad 1: Net-(D1-A) -> GND
- R2 pad 2: /Obstruction_5V -> Net-(D1-K)
- R3 pad 1: /Obstruction_3V -> Net-(Q1-C)
- R3 pad 2: +3V3 -> Net-(Q2-B)
- R4 pad 1: /ObstructionObserved_3V -> Net-(Q1-C)
- R4 pad 2: /Obstruction_3V -> +5V
- R5 pad 1: /Obstruction_5V -> Net-(Q2-C)
- R5 pad 2: /Obstruction -> +5V
- U2 pad 10: unconnected-(U1-A8-Pad10) -> GND
- U2 pad 21: /Obstruction_3V -> /ObstructionObserved_3V
- U2 pad 3: /Obstruction_5V -> /ObstructionObserved_5V
- U2 pad 9: unconnected-(U1-A7-Pad9) -> GND
Routing:
- net /Obstruction_5V: track 20.1 -> 0.00 mm
- net Net-(Q2-B): track 0.00 -> 10.6 mm
- net /Obstruction_3V: track 9.23 -> 0.00 mm
- net /ObstructionObserved_5V: track 0.00 -> 8.43 mm
- net Net-(Q2-C): track 0.00 -> 8.29 mm
- net GND: track 21.9 -> 30.1 mm, vias 13 -> 17
- net Net-(D1-K): track 1.50 -> 9.52 mm
- net +5V: track 82.6 -> 90.4 mm, vias 3 -> 4
- net /ObstructionObserved_3V: track 4.56 -> 10.8 mm
- net Net-(Q1-C): track 0.00 -> 5.71 mm
- net /Obstruction: track 34.1 -> 28.9 mm
- net Net-(D1-A): track 3.40 -> 0.00 mm
- net +3V3: track 67.6 -> 66.1 mm
Other:
- board text added: "Mtr Closing"
- board text added: "Mtr Opening"
- board text removed: "Relay2"
- board text removed: "Relay3"
