File: pcb/200280rB.kicad_sch (KiCad schematic)
At the start: 26 parts, among them J1 ScrewTerms, Q1 SI2304BDS-T1-GE3, Q2 SI2304BDS-T1-GE3, Q3 SI2304BDS-T1-GE3, U1 SN74AVC8T245PW, U2 XIAO-ESP32-S3-SMD, U3 OKI-78SR-5/1.5-W36-C

Commit message: as purchased revision B
Parts:
- removed C1: 1uF, Capacitor_SMD:C_0603_1608Metric, symbol Device:C
- removed D1, D2, D3: MMBD4448HTS, Package_TO_SOT_SMD:SOT-523, symbol Device:D_Dual_Series_AKC
- removed Q1: SI2304BDS-T1-GE3, Package_TO_SOT_SMD:SOT-23, symbol Device:Q_NMOS_GSD
- added C3: 1uF, Capacitor_SMD:C_0603_1608Metric, symbol Device:C
- added D1: 5.1V, Diode_SMD:D_SOD-323_HandSoldering, symbol Device:D_Zener
- added Q1, Q2: MMBT3904, Package_TO_SOT_SMD:SOT-23-3, symbol Device:Q_NPN_BEC
- R1: value 100K -> 10K
- R2: value DNP -> 4K7; now fitted
- R3: value 100K -> 2K
- R4: value 680R -> 20K
- R5: value 680R -> 100K
- R6: value 120R -> 680R
- renumbered C3 to C1, H4 to H2, Q2 to Q4, R7 to R10, R10 to R7, R9 to R8, R8 to R9, U3 to U1, U1 to U2, U2 to U3
Connections:
- net +3V3: no longer R3.2
- net +5V: now also R4.2, R5.2; no longer R1.2
- net GND: now also R2.1, U2.10 (A8), U2.9 (A7), C3.2, D1.2 (A), Q1.2 (E), Q2.2 (E)
- net Obstruction: now also R1.2; no longer R5.2
- net ObstructionObserved_3V: now also U2.21 (B1); no longer R4.1
- net at R3.1: now also R4.1, Q1.3 (C); no longer R4.2
- net at R6.2: now also R5.1, C3.1, Q2.3 (C)
- net Obstruction_3V renamed ObstructionObserved_5V
- net ObstructionObserved_5V: now also U2.3 (A1); no longer U2.21 (B1)
- net Obstruction_5V: no longer names the net of R1.1, R2.2
- net Obstruction_5V: now also D1.1 (K), Q1.1 (B); no longer R5.1, U2.3 (A1)
- net Relay2_ renamed Relay2_Motor_Closing
- net Relay2__3V renamed Relay2_Motor_Closing_3V
- net Relay3_ renamed Relay3_Motor_Opening
- net Relay3__3V renamed Relay3_Motor_Opening_3V
- net Return?: no longer names the net of J1.2 (Pin_2)
- new net: Q2.1 (B), R3.2
Other:
- note added: "Output: 0-5V Low = NoObstruction High = Obstruction"
- note added: "Screw Terminals Wires soldered directly to microcontroller pins on Garage Door Opener Main PCB Logic: EndStopOpen = 5V when not active; 0V when Active EndStopClosed = 5V when not active; 0V when Active Relay1_Light = 5V when not active; 0V when Active Relay2_Motor_Closing = 5V when not active; 0V when Active Relay3_Motor_Opening = 5V when not active; 0V when Active Obstruction = 16V when obstruct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"
- note removed: "Measured +6VDC MAX"
- note removed: "Output: 0-3V3 Low = NoObstruction High = Obstruction"
- note removed: "Screw Terminals Wires soldered directly to microcontroller pins on Garage Door Opener Main PCB Logic: EndStopOpen = 5V when not active; 0V when Active EndStopClosed = 5V when not active; 0V when Active Relay1_Light = 5V when not active; 0V when Active Relay2_ = 5V when not active; 0V when Active Relay3_ = 5V when not active; 0V when Active Obstruction = 16V when obstruction; low pulses when NoObs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"
- moved on the sheet: C1, C2, U2
